File: Example/ESP-12EF-breakout_board/breakout_board.sch (EAGLE design)
At the start: 4 parts, among them IC1 ESP-12E/F

Commit message: adding example
Parts:
- removed C1: (no value), resistor:C-EUC0805
Connections:
- removed net +3V3: C1.1, IC1.VCC
- net GND: no longer C1.2
- net VCC: now also IC1.VCC
Changed lines of the file:
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@@
 <part name="GND1" library="supply1" deviceset="GND" device=""/>
 <part name="+3V1" library="supply1" deviceset="+3V3" device=""/>
-<part name="C1" library="resistor" deviceset="C-EU" device="C0805"/>
-<part name="GND2" library="supply1" deviceset="GND" device=""/>
 <part name="JP2" library="pinhead" deviceset="PINHD-1X11" device=""/>
 <part name="FRAME1" library="frames" deviceset="A5L-LOC" device=""/>
@@
 </plain>
 <instances>
-<instance part="IC1" gate="G$1" x="67.31" y="73.66"/>
+<instance part="IC1" gate="G$1" x="59.69" y="68.58"/>
 <instance part="JP1" gate="A" x="143.51" y="76.2"/>
 <instance part="GND1" gate="1" x="90.17" y="44.45"/>
 <instance part="+3V1" gate="G$1" x="26.67" y="53.34"/>
-<instance part="C1" gate="G$1" x="26.67" y="40.64"/>
-<instance part="GND2" gate="1" x="26.67" y="33.02"/>
 <instance part="JP2" gate="A" x="168.91" y="76.2"/>
 <instance part="FRAME1" gate="G$1" x="1.27" y="0"/>
@@
 <net name="GND" class="0">
 <segment>
-<pinref part="C1" gate="G$1" pin="2"/>
-<pinref part="GND2" gate="1" pin="GND"/>
-</segment>
-<segment>
 <pinref part="IC1" gate="G$1" pin="GND"/>
 <pinref part="GND1" gate="1" pin="GND"/>
@@
 </segment>
 </net>
-<net name="+3V3" class="0">
-<segment>
-<pinref part="C1" gate="G$1" pin="1"/>
-<pinref part="+3V1" gate="G$1" pin="+3V3"/>
-<wire x1="26.67" y1="50.8" x2="26.67" y2="46.99" width="0.1524" layer="91"/>
-<wire x1="26.67" y1="46.99" x2="26.67" y2="43.18" width="0.1524" layer="91"/>
-<wire x1="26.67" y1="46.99" x2="31.75" y2="46.99" width="0.1524" layer="91"/>
-<wire x1="31.75" y1="46.99" x2="31.75" y2="53.34" width="0.1524" layer="91"/>
-<junction x="26.67" y="46.99"/>
-<pinref part="IC1" gate="G$1" pin="VCC"/>
-<wire x1="31.75" y1="53.34" x2="34.29" y2="53.34" width="0.1524" layer="91"/>
-</segment>
-</net>
 <net name="CS0" class="0">
 <segment>
@@
 <label x="128.27" y="71.12" size="1.778" layer="95"/>
 </segment>
-</net>
+<segment>
+<pinref part="+3V1" gate="G$1" pin="+3V3"/>
+<wire x1="26.67" y1="50.8" x2="26.67" y2="46.99" width="0.1524" layer="91"/>
+<wire x1="26.67" y1="46.99" x2="31.75" y2="46.99" width="0.1524" layer="91"/>
+<wire x1="31.75" y1="46.99" x2="31.75" y2="53.34" width="0.1524" layer="91"/>
+<pinref part="IC1" gate="G$1" pin="VCC"/>
+<wire x1="31.75" y1="53.34" x2="34.29" y2="53.34" width="0.1524" layer="91"/>
+</segment>
+</net>
